Commit message: removed absolute paths from URDF files and added `FileUriResolver` for resolving file paths; updated episode executor with support for fixed objects and path resolver options

File: resources/multiverse_episodes/icub_montessori_no_hands/models/montessori_object_2.urdf (robot description, URDF)
Before this commit: robot montessori_object_2, 1 links, 0 joints
Links:
- link montessori_object_2: geometry collision mesh filename=file://montessori_object_1/meshes/stl/montessori_object_2_M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 scale=1.0 1.0 1.0

File: resources/multiverse_episodes/icub_montessori_no_hands/models/scene.urdf (robot description, URDF)
Before this commit: robot iCub_with_montessori_toys_2, 16 links, 15 joints
Links:
- link montessori_box: geometry collision box size=0.0020000000949949026 0.257999986410141 0.06400000303983688; collision box size=0.004999999888241291 0.026000000536441803 0.008000000379979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
- link montessori_drawer_1: geometry collision box size=0.004999999888241291 0.07199999690055847 0.05999999865889549; collision box size=0.00800000037997961 0.0820000022649765 0.05999999865889549
- link montessori_drawer_1_handle: geometry collision cylinder length=0.014999999664723873 radius=0.00800000037997961; collision sphere radius=0.004999999888241291
- link montessori_drawer_2: geometry collision box size=0.004999999888241291 0.07199999690055847 0.05999999865889549; collision box size=0.00800000037997961 0.0820000022649765 0.05999999865889549
- link montessori_drawer_2_handle: geometry collision cylinder length=0.014999999664723873 radius=0.00800000037997961; collision sphere radius=0.004999999888241291
- link montessori_drawer_3: geometry collision box size=0.004999999888241291 0.07199999690055847 0.05999999865889549; collision box size=0.00800000037997961 0.0820000022649765 0.05999999865889549
- link montessori_drawer_3_handle: geometry collision cylinder length=0.014999999664723873 radius=0.00800000037997961; collision sphere radius=0.004999999888241291
- link triangle_hole: geometry collision mesh filename=file://scene/meshes/stl/montessori_object_2_MontessoriObjec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 scale=0.8 0.8 0.02
