Commit message: Task T3: the G1 finds the loose bolt and brings the torque tool
Tool rack at the rear of the nacelle, tool tray on the -Y girder, a
technician placeholder (scenario extras), scenario bring_the_tool and
scripts/g1_bring_the_tool.py: shrink disc torque-marking check, pick up
the tool case at the rack, carry it along the walkway, place it on the
tray next to the technician. Recorded for CRAMERA (windturbine_g1_t3).

Co-Authored-By: Claude Opus 5.5 <noreply@anthropic.com>
Claude-Session: https://claude.ai/code/session_01BXKsjsesbT14QvbqkbYZ34

File: urdf/scenarios/bring_the_tool.urdf (robot description, URDF)
Before this commit: robot windturbine, 98 links, 97 joints
Links:
- removed link gearbox_fault_oil_puddle
- removed link gearbox_fault_oil_streak
- removed link generator_fault_carbon_dust
- removed link generator_fault_terminal_heat
- removed link hydraulic_fault_leak
- removed link main_bearing_fault_grease_leak
- removed link main_shaft_fault_fretting
- added link technician, mass 1.0; collision box size=0.44 0.28 1.78; visual mesh filename=package://windturbine_model/models/systems/technician.obj
- link converter_status_light: geometry visual mesh filename=package://windturbine_model/models/systems/status_light_ok_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
- link cooling_level: geometry visual mesh filename=package://windturbine_model/models/systems/coolant_level_ok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
- link fast_shaft_brake_disc: geometry collision cylinder length=0.06 radius=0.45; visual mesh filename=package://windturbine_model/models/generator/brake_disc_ok.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
- link fast_shaft_coupling: geometry collision cylinder length=0.55 radius=0.3; visual mesh filename=package://windturbine_model/models/generator/coupling_ok.obj
- link fire_extinguisher: geometry visual mesh filename=package://windturbine_model/models/systems/extinguisher_pre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
- link gearbox_bushing_left: geometry visual mesh filename=package://windturbine_model/models/gearbox/bushing_left_ok.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
- link gearbox_cover_bolts: geometry visual mesh filename=package://windturbine_model/models/gearbox/cover_bolts_ok.o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
- link gearbox_sight_glass: geometry visual mesh filename=package://windturbine_model/models/gearbox/sight_glass_ok.o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
Joints:
- removed joint gearbox_fault_oil_puddle_joint
- removed joint gearbox_fault_oil_streak_joint
- removed joint generator_fault_carbon_dust_joint
- removed joint generator_fault_terminal_heat_joint
- removed joint hydraulic_fault_leak_joint
- removed joint main_bearing_fault_grease_leak_joint
- removed joint main_shaft_fault_fretting_joint
- added joint technician_joint: type fixed, parent nacelle, child technician, origin xyz=2 -1.7 0 rpy=0 0 0

File: urdf/scenarios/outside_all_faults.urdf (robot description, URDF)
Before this commit: robot windturbine, 96 links, 95 joints
Links:
- added link tool_rack, mass 1.0; collision box size=0.6 0.02 1.3; collision box size=0.6 0.32 0.03
- added link tool_tray, mass 1.0; collision box size=0.4 0.27 0.025; visual mesh filename=package://windturbine_model/models/systems/tool_tray.obj
Joints:
- added joint tool_rack_joint: type fixed, parent nacelle, child tool_rack, origin xyz=0 0 0 rpy=0 0 0
- added joint tool_tray_joint: type fixed, parent nacelle, child tool_tray, origin xyz=0 0 0 rpy=0 0 0

File: urdf/windturbine.urdf (robot description, URDF)
Before this commit: robot windturbine, 89 links, 88 joints
Links:
- added link tool_rack, mass 1.0; collision box size=0.6 0.02 1.3; collision box size=0.6 0.32 0.03
- added link tool_tray, mass 1.0; collision box size=0.4 0.27 0.025; visual mesh filename=package://windturbine_model/models/systems/tool_tray.obj
Joints:
- added joint tool_rack_joint: type fixed, parent nacelle, child tool_rack, origin xyz=0 0 0 rpy=0 0 0
- added joint tool_tray_joint: type fixed, parent nacelle, child tool_tray, origin xyz=0 0 0 rpy=0 0 0
