Commit message: G1 inspection rounds T1/T2, recorded for CRAMERA
scripts/g1_inspection_round.py drives the Unitree G1 through a zone's
inspection points (ground around the tower, nacelle walkway), aims its
D435 along the optical x axis (CRAM's annotation declares z), aims below
shallow targets so they land in the image, and reports the ground-truth
findings. scripts/finish_recording.py tidies cramera-onboard bundles
(robot naming, GLB materials, camera, nacelle cover). Plinth collision as
boxes so the route planner sees a round footprint; the old T0 script is
folded into the round (--points tower_inspect_door).

Co-Authored-By: Claude Opus 5.5 <noreply@anthropic.com>
Claude-Session: https://claude.ai/code/session_01BXKsjsesbT14QvbqkbYZ34

File: urdf/scenarios/after_maintenance.urdf (robot description, URDF)
Before this commit: robot windturbine, 89 links, 88 joints
Links:
- link foundation: geometry collision box size=1.16228 1.04689 0.24; collision box size=1.16228 1.04689 0.24
Joints:
- joint tower_inspect_base_coating_joint: origin xyz=1.67276 -2.47997 1.3 rpy=0 0 0 -> xyz=1.67385 -2.48159 0.6 rpy=0 0 0
- joint tower_inspect_door_joint: origin xyz=0 -3.04233 1.96 rpy=0 0 0 -> xyz=0 -3.04233 1.31 rpy=0 0 0

File: urdf/scenarios/blade_damage.urdf (robot description, URDF)
Before this commit: robot windturbine, 92 links, 91 joints
Links:
- link foundation: geometry collision box size=1.16228 1.04689 0.24; collision box size=1.16228 1.04689 0.24
Joints:
- joint tower_inspect_base_coating_joint: origin xyz=1.67276 -2.47997 1.3 rpy=0 0 0 -> xyz=1.67385 -2.48159 0.6 rpy=0 0 0
- joint tower_inspect_door_joint: origin xyz=0 -3.04233 1.96 rpy=0 0 0 -> xyz=0 -3.04233 1.31 rpy=0 0 0

File: urdf/scenarios/gearbox_all_faults.urdf (robot description, URDF)
Before this commit: robot windturbine, 91 links, 90 joints
Links:
- link foundation: geometry collision box size=1.16228 1.04689 0.24; collision box size=1.16228 1.04689 0.24
Joints:
- joint tower_inspect_base_coating_joint: origin xyz=1.67276 -2.47997 1.3 rpy=0 0 0 -> xyz=1.67385 -2.48159 0.6 rpy=0 0 0
- joint tower_inspect_door_joint: origin xyz=0 -3.04233 1.96 rpy=0 0 0 -> xyz=0 -3.04233 1.31 rpy=0 0 0

File: urdf/scenarios/gearbox_seal_leak.urdf (robot description, URDF)
Before this commit: robot windturbine, 91 links, 90 joints
Links:
- link foundation: geometry collision box size=1.16228 1.04689 0.24; collision box size=1.16228 1.04689 0.24
Joints:
- joint tower_inspect_base_coating_joint: origin xyz=1.67276 -2.47997 1.3 rpy=0 0 0 -> xyz=1.67385 -2.48159 0.6 rpy=0 0 0
- joint tower_inspect_door_joint: origin xyz=0 -3.04233 1.96 rpy=0 0 0 -> xyz=0 -3.04233 1.31 rpy=0 0 0

File: urdf/scenarios/generator_all_faults.urdf (robot description, URDF)
Before this commit: robot windturbine, 91 links, 90 joints
Links:
- link foundation: geometry collision box size=1.16228 1.04689 0.24; collision box size=1.16228 1.04689 0.24
Joints:
- joint tower_inspect_base_coating_joint: origin xyz=1.67276 -2.47997 1.3 rpy=0 0 0 -> xyz=1.67385 -2.48159 0.6 rpy=0 0 0
- joint tower_inspect_door_joint: origin xyz=0 -3.04233 1.96 rpy=0 0 0 -> xyz=0 -3.04233 1.31 rpy=0 0 0

File: urdf/scenarios/main_shaft_all_faults.urdf (robot description, URDF)
Before this commit: robot windturbine, 91 links, 90 joints
Links:
- link foundation: geometry collision box size=1.16228 1.04689 0.24; collision box size=1.16228 1.04689 0.24
Joints:
- joint tower_inspect_base_coating_joint: origin xyz=1.67276 -2.47997 1.3 rpy=0 0 0 -> xyz=1.67385 -2.48159 0.6 rpy=0 0 0
- joint tower_inspect_door_joint: origin xyz=0 -3.04233 1.96 rpy=0 0 0 -> xyz=0 -3.04233 1.31 rpy=0 0 0

File: urdf/scenarios/nacelle_all_faults.urdf (robot description, URDF)
Before this commit: robot windturbine, 96 links, 95 joints
Links:
- link foundation: geometry collision box size=1.16228 1.04689 0.24; collision box size=1.16228 1.04689 0.24
Joints:
- joint tower_inspect_base_coating_joint: origin xyz=1.67276 -2.47997 1.3 rpy=0 0 0 -> xyz=1.67385 -2.48159 0.6 rpy=0 0 0
- joint tower_inspect_door_joint: origin xyz=0 -3.04233 1.96 rpy=0 0 0 -> xyz=0 -3.04233 1.31 rpy=0 0 0

File: urdf/scenarios/nacelle_systems_faults.urdf (robot description, URDF)
Before this commit: robot windturbine, 90 links, 89 joints
Links:
- link foundation: geometry collision box size=1.16228 1.04689 0.24; collision box size=1.16228 1.04689 0.24
Joints:
- joint tower_inspect_base_coating_joint: origin xyz=1.67276 -2.47997 1.3 rpy=0 0 0 -> xyz=1.67385 -2.48159 0.6 rpy=0 0 0
- joint tower_inspect_door_joint: origin xyz=0 -3.04233 1.96 rpy=0 0 0 -> xyz=0 -3.04233 1.31 rpy=0 0 0

File: urdf/scenarios/outside_all_faults.urdf (robot description, URDF)
Before this commit: robot windturbine, 96 links, 95 joints
Links:
- link foundation: geometry collision box size=1.16228 1.04689 0.24; collision box size=1.16228 1.04689 0.24
Joints:
- joint tower_inspect_base_coating_joint: origin xyz=1.67276 -2.47997 1.3 rpy=0 0 0 -> xyz=1.67385 -2.48159 0.6 rpy=0 0 0
- joint tower_inspect_door_joint: origin xyz=0 -3.04233 1.96 rpy=0 0 0 -> xyz=0 -3.04233 1.31 rpy=0 0 0

File: urdf/scenarios/outside_ground.urdf (robot description, URDF)
Before this commit: robot windturbine, 92 links, 91 joints
Links:
- link foundation: geometry collision box size=1.16228 1.04689 0.24; collision box size=1.16228 1.04689 0.24
Joints:
- joint tower_inspect_base_coating_joint: origin xyz=1.67276 -2.47997 1.3 rpy=0 0 0 -> xyz=1.67385 -2.48159 0.6 rpy=0 0 0
- joint tower_inspect_door_joint: origin xyz=0 -3.04233 1.96 rpy=0 0 0 -> xyz=0 -3.04233 1.31 rpy=0 0 0

File: urdf/windturbine.urdf (robot description, URDF)
Before this commit: robot windturbine, 89 links, 88 joints
Links:
- link foundation: geometry collision box size=1.16228 1.04689 0.24; collision box size=1.16228 1.04689 0.24
Joints:
- joint tower_inspect_base_coating_joint: origin xyz=1.67276 -2.47997 1.3 rpy=0 0 0 -> xyz=1.67385 -2.48159 0.6 rpy=0 0 0
- joint tower_inspect_door_joint: origin xyz=0 -3.04233 1.96 rpy=0 0 0 -> xyz=0 -3.04233 1.31 rpy=0 0 0
