Commit message: T6: G1 flange bolt check up the tower, with tightness ratio and actions
- 364 flange bolts (132 M42, 132 M42, 100 M36; estimated sizes) with torque
  markings on the nuts; faults turn markings on flange 2 (one nut run off) and 3.
- turbine/bolts.py: preload from the marking offset (nut turn to full preload from
  bolt and joint stiffness), ACP RP 401 thresholds, actions per flange.
- scripts/g1_tower_bolts.py: lift stops at each rest platform, a ring of
  standpoints per flange, visibility per nut (field of view, range, angle, lift car,
  flange edge), ride down, walk out; report to reports/tower_bolt_check.{md,json}.
- Lift joint headroom below 0; video playback speed; tower cutaway also cuts bolts.
- Gallery: bolt check section with the report table and video.

Co-Authored-By: Claude Opus 5.5 <noreply@anthropic.com>
Claude-Session: https://claude.ai/code/session_01BXKsjsesbT14QvbqkbYZ34

File: urdf/scenarios/after_maintenance.urdf (robot description, URDF)
Before this commit: robot windturbine, 105 links, 104 joints
Links:
- added link flange_1_bolts, mass 1.0; visual mesh filename=package://windturbine_model/models/tower_interior/flange_1_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
- added link flange_2_bolts, mass 1.0; visual mesh filename=package://windturbine_model/models/tower_interior/flange_2_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
- added link flange_3_bolts, mass 1.0; visual mesh filename=package://windturbine_model/models/tower_interior/flange_3_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
- added link tower_inspect_flange_1, mass 1.0
- added link tower_inspect_flange_2, mass 1.0
- added link tower_inspect_flange_3, mass 1.0
Joints:
- added joint flange_1_bolts_joint: type fixed, parent tower_section_1, child flange_1_bolts, origin xyz=0 0 0 rpy=0 0 0
- added joint flange_2_bolts_joint: type fixed, parent tower_section_2, child flange_2_bolts, origin xyz=0 0 0 rpy=0 0 0
- added joint flange_3_bolts_joint: type fixed, parent tower_section_3, child flange_3_bolts, origin xyz=0 0 0 rpy=0 0 0
- added joint tower_inspect_flange_1_joint: type fixed, parent tower_section_1, child tower_inspect_flange_1, origin xyz=2.77203 0 21.446 rpy=0 0 0
- added joint tower_inspect_flange_2_joint: type fixed, parent tower_section_2, child tower_inspect_flange_2, origin xyz=1.39448 2.41531 32.246 rpy=0 0 0
- added joint tower_inspect_flange_3_joint: type fixed, parent tower_section_3, child tower_inspect_flange_3, origin xyz=-3.70381e-16 -2.01626 32.2495 rpy=0 0 0
- joint service_lift_joint: limit lower=0.0 upper=105.66000000000001 effort=100 velocity=4.0 -> lower=-0.1 upper=105.66000000000001 effort=100 velocity=4.0
- joint tower_inspect_cable_loop_joint: origin xyz=0.139 -0.001 19.27 rpy=0 0 0 -> xyz=0.099 0.159 19.27 rpy=0 0 0

File: urdf/scenarios/blade_damage.urdf (robot description, URDF)
Before this commit: robot windturbine, 108 links, 107 joints
Links:
- added link flange_1_bolts, mass 1.0; visual mesh filename=package://windturbine_model/models/tower_interior/flange_1_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
- added link flange_2_bolts, mass 1.0; visual mesh filename=package://windturbine_model/models/tower_interior/flange_2_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
- added link flange_3_bolts, mass 1.0; visual mesh filename=package://windturbine_model/models/tower_interior/flange_3_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
- added link tower_inspect_flange_1, mass 1.0
- added link tower_inspect_flange_2, mass 1.0
- added link tower_inspect_flange_3, mass 1.0
Joints:
- added joint flange_1_bolts_joint: type fixed, parent tower_section_1, child flange_1_bolts, origin xyz=0 0 0 rpy=0 0 0
- added joint flange_2_bolts_joint: type fixed, parent tower_section_2, child flange_2_bolts, origin xyz=0 0 0 rpy=0 0 0
- added joint flange_3_bolts_joint: type fixed, parent tower_section_3, child flange_3_bolts, origin xyz=0 0 0 rpy=0 0 0
- added joint tower_inspect_flange_1_joint: type fixed, parent tower_section_1, child tower_inspect_flange_1, origin xyz=2.77203 0 21.446 rpy=0 0 0
- added joint tower_inspect_flange_2_joint: type fixed, parent tower_section_2, child tower_inspect_flange_2, origin xyz=1.39448 2.41531 32.246 rpy=0 0 0
- added joint tower_inspect_flange_3_joint: type fixed, parent tower_section_3, child tower_inspect_flange_3, origin xyz=-3.70381e-16 -2.01626 32.2495 rpy=0 0 0
- joint service_lift_joint: limit lower=0.0 upper=105.66000000000001 effort=100 velocity=4.0 -> lower=-0.1 upper=105.66000000000001 effort=100 velocity=4.0
- joint tower_inspect_cable_loop_joint: origin xyz=0.139 -0.001 19.27 rpy=0 0 0 -> xyz=0.099 0.159 19.27 rpy=0 0 0

File: urdf/scenarios/bring_the_tool.urdf (robot description, URDF)
Before this commit: robot windturbine, 106 links, 105 joints
Links:
- added link flange_1_bolts, mass 1.0; visual mesh filename=package://windturbine_model/models/tower_interior/flange_1_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
- added link flange_2_bolts, mass 1.0; visual mesh filename=package://windturbine_model/models/tower_interior/flange_2_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
- added link flange_3_bolts, mass 1.0; visual mesh filename=package://windturbine_model/models/tower_interior/flange_3_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
- added link tower_inspect_flange_1, mass 1.0
- added link tower_inspect_flange_2, mass 1.0
- added link tower_inspect_flange_3, mass 1.0
Joints:
- added joint flange_1_bolts_joint: type fixed, parent tower_section_1, child flange_1_bolts, origin xyz=0 0 0 rpy=0 0 0
- added joint flange_2_bolts_joint: type fixed, parent tower_section_2, child flange_2_bolts, origin xyz=0 0 0 rpy=0 0 0
- added joint flange_3_bolts_joint: type fixed, parent tower_section_3, child flange_3_bolts, origin xyz=0 0 0 rpy=0 0 0
- added joint tower_inspect_flange_1_joint: type fixed, parent tower_section_1, child tower_inspect_flange_1, origin xyz=2.77203 0 21.446 rpy=0 0 0
- added joint tower_inspect_flange_2_joint: type fixed, parent tower_section_2, child tower_inspect_flange_2, origin xyz=1.39448 2.41531 32.246 rpy=0 0 0
- added joint tower_inspect_flange_3_joint: type fixed, parent tower_section_3, child tower_inspect_flange_3, origin xyz=-3.70381e-16 -2.01626 32.2495 rpy=0 0 0
- joint service_lift_joint: limit lower=0.0 upper=105.66000000000001 effort=100 velocity=4.0 -> lower=-0.1 upper=105.66000000000001 effort=100 velocity=4.0
- joint tower_inspect_cable_loop_joint: origin xyz=0.139 -0.001 19.27 rpy=0 0 0 -> xyz=0.099 0.159 19.27 rpy=0 0 0

File: urdf/scenarios/gearbox_all_faults.urdf (robot description, URDF)
Before this commit: robot windturbine, 107 links, 106 joints
Links:
- added link flange_1_bolts, mass 1.0; visual mesh filename=package://windturbine_model/models/tower_interior/flange_1_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
- added link flange_2_bolts, mass 1.0; visual mesh filename=package://windturbine_model/models/tower_interior/flange_2_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
- added link flange_3_bolts, mass 1.0; visual mesh filename=package://windturbine_model/models/tower_interior/flange_3_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
- added link tower_inspect_flange_1, mass 1.0
- added link tower_inspect_flange_2, mass 1.0
- added link tower_inspect_flange_3, mass 1.0
Joints:
- added joint flange_1_bolts_joint: type fixed, parent tower_section_1, child flange_1_bolts, origin xyz=0 0 0 rpy=0 0 0
- added joint flange_2_bolts_joint: type fixed, parent tower_section_2, child flange_2_bolts, origin xyz=0 0 0 rpy=0 0 0
- added joint flange_3_bolts_joint: type fixed, parent tower_section_3, child flange_3_bolts, origin xyz=0 0 0 rpy=0 0 0
- added joint tower_inspect_flange_1_joint: type fixed, parent tower_section_1, child tower_inspect_flange_1, origin xyz=2.77203 0 21.446 rpy=0 0 0
- added joint tower_inspect_flange_2_joint: type fixed, parent tower_section_2, child tower_inspect_flange_2, origin xyz=1.39448 2.41531 32.246 rpy=0 0 0
- added joint tower_inspect_flange_3_joint: type fixed, parent tower_section_3, child tower_inspect_flange_3, origin xyz=-3.70381e-16 -2.01626 32.2495 rpy=0 0 0
- joint service_lift_joint: limit lower=0.0 upper=105.66000000000001 effort=100 velocity=4.0 -> lower=-0.1 upper=105.66000000000001 effort=100 velocity=4.0
- joint tower_inspect_cable_loop_joint: origin xyz=0.139 -0.001 19.27 rpy=0 0 0 -> xyz=0.099 0.159 19.27 rpy=0 0 0

File: urdf/scenarios/gearbox_seal_leak.urdf (robot description, URDF)
Before this commit: robot windturbine, 107 links, 106 joints
Links:
- added link flange_1_bolts, mass 1.0; visual mesh filename=package://windturbine_model/models/tower_interior/flange_1_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
- added link flange_2_bolts, mass 1.0; visual mesh filename=package://windturbine_model/models/tower_interior/flange_2_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
- added link flange_3_bolts, mass 1.0; visual mesh filename=package://windturbine_model/models/tower_interior/flange_3_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
- added link tower_inspect_flange_1, mass 1.0
- added link tower_inspect_flange_2, mass 1.0
- added link tower_inspect_flange_3, mass 1.0
Joints:
- added joint flange_1_bolts_joint: type fixed, parent tower_section_1, child flange_1_bolts, origin xyz=0 0 0 rpy=0 0 0
- added joint flange_2_bolts_joint: type fixed, parent tower_section_2, child flange_2_bolts, origin xyz=0 0 0 rpy=0 0 0
- added joint flange_3_bolts_joint: type fixed, parent tower_section_3, child flange_3_bolts, origin xyz=0 0 0 rpy=0 0 0
- added joint tower_inspect_flange_1_joint: type fixed, parent tower_section_1, child tower_inspect_flange_1, origin xyz=2.77203 0 21.446 rpy=0 0 0
- added joint tower_inspect_flange_2_joint: type fixed, parent tower_section_2, child tower_inspect_flange_2, origin xyz=1.39448 2.41531 32.246 rpy=0 0 0
- added joint tower_inspect_flange_3_joint: type fixed, parent tower_section_3, child tower_inspect_flange_3, origin xyz=-3.70381e-16 -2.01626 32.2495 rpy=0 0 0
- joint service_lift_joint: limit lower=0.0 upper=105.66000000000001 effort=100 velocity=4.0 -> lower=-0.1 upper=105.66000000000001 effort=100 velocity=4.0
- joint tower_inspect_cable_loop_joint: origin xyz=0.139 -0.001 19.27 rpy=0 0 0 -> xyz=0.099 0.159 19.27 rpy=0 0 0

File: urdf/scenarios/hoist_access.urdf (robot description, URDF)
Before this commit: robot windturbine, 105 links, 104 joints
Links:
- added link flange_1_bolts, mass 1.0; visual mesh filename=package://windturbine_model/models/tower_interior/flange_1_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
- added link flange_2_bolts, mass 1.0; visual mesh filename=package://windturbine_model/models/tower_interior/flange_2_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
- added link flange_3_bolts, mass 1.0; visual mesh filename=package://windturbine_model/models/tower_interior/flange_3_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
- added link tower_inspect_flange_1, mass 1.0
- added link tower_inspect_flange_2, mass 1.0
- added link tower_inspect_flange_3, mass 1.0
Joints:
- added joint flange_1_bolts_joint: type fixed, parent tower_section_1, child flange_1_bolts, origin xyz=0 0 0 rpy=0 0 0
- added joint flange_2_bolts_joint: type fixed, parent tower_section_2, child flange_2_bolts, origin xyz=0 0 0 rpy=0 0 0
- added joint flange_3_bolts_joint: type fixed, parent tower_section_3, child flange_3_bolts, origin xyz=0 0 0 rpy=0 0 0
- added joint tower_inspect_flange_1_joint: type fixed, parent tower_section_1, child tower_inspect_flange_1, origin xyz=2.77203 0 21.446 rpy=0 0 0
- added joint tower_inspect_flange_2_joint: type fixed, parent tower_section_2, child tower_inspect_flange_2, origin xyz=1.39448 2.41531 32.246 rpy=0 0 0
- added joint tower_inspect_flange_3_joint: type fixed, parent tower_section_3, child tower_inspect_flange_3, origin xyz=-3.70381e-16 -2.01626 32.2495 rpy=0 0 0
- joint service_lift_joint: limit lower=0.0 upper=105.66000000000001 effort=100 velocity=4.0 -> lower=-0.1 upper=105.66000000000001 effort=100 velocity=4.0
- joint tower_inspect_cable_loop_joint: origin xyz=0.139 -0.001 19.27 rpy=0 0 0 -> xyz=0.099 0.159 19.27 rpy=0 0 0

File: urdf/scenarios/main_shaft_all_faults.urdf (robot description, URDF)
Before this commit: robot windturbine, 107 links, 106 joints
Links:
- added link flange_1_bolts, mass 1.0; visual mesh filename=package://windturbine_model/models/tower_interior/flange_1_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
- added link flange_2_bolts, mass 1.0; visual mesh filename=package://windturbine_model/models/tower_interior/flange_2_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
- added link flange_3_bolts, mass 1.0; visual mesh filename=package://windturbine_model/models/tower_interior/flange_3_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
- added link tower_inspect_flange_1, mass 1.0
- added link tower_inspect_flange_2, mass 1.0
- added link tower_inspect_flange_3, mass 1.0
Joints:
- added joint flange_1_bolts_joint: type fixed, parent tower_section_1, child flange_1_bolts, origin xyz=0 0 0 rpy=0 0 0
- added joint flange_2_bolts_joint: type fixed, parent tower_section_2, child flange_2_bolts, origin xyz=0 0 0 rpy=0 0 0
- added joint flange_3_bolts_joint: type fixed, parent tower_section_3, child flange_3_bolts, origin xyz=0 0 0 rpy=0 0 0
- added joint tower_inspect_flange_1_joint: type fixed, parent tower_section_1, child tower_inspect_flange_1, origin xyz=2.77203 0 21.446 rpy=0 0 0
- added joint tower_inspect_flange_2_joint: type fixed, parent tower_section_2, child tower_inspect_flange_2, origin xyz=1.39448 2.41531 32.246 rpy=0 0 0
- added joint tower_inspect_flange_3_joint: type fixed, parent tower_section_3, child tower_inspect_flange_3, origin xyz=-3.70381e-16 -2.01626 32.2495 rpy=0 0 0
- joint service_lift_joint: limit lower=0.0 upper=105.66000000000001 effort=100 velocity=4.0 -> lower=-0.1 upper=105.66000000000001 effort=100 velocity=4.0
- joint tower_inspect_cable_loop_joint: origin xyz=0.139 -0.001 19.27 rpy=0 0 0 -> xyz=0.099 0.159 19.27 rpy=0 0 0

File: urdf/scenarios/nacelle_all_faults.urdf (robot description, URDF)
Before this commit: robot windturbine, 112 links, 111 joints
Links:
- added link flange_1_bolts, mass 1.0; visual mesh filename=package://windturbine_model/models/tower_interior/flange_1_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
- added link flange_2_bolts, mass 1.0; visual mesh filename=package://windturbine_model/models/tower_interior/flange_2_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
- added link flange_3_bolts, mass 1.0; visual mesh filename=package://windturbine_model/models/tower_interior/flange_3_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
- added link tower_inspect_flange_1, mass 1.0
- added link tower_inspect_flange_2, mass 1.0
- added link tower_inspect_flange_3, mass 1.0
Joints:
- added joint flange_1_bolts_joint: type fixed, parent tower_section_1, child flange_1_bolts, origin xyz=0 0 0 rpy=0 0 0
- added joint flange_2_bolts_joint: type fixed, parent tower_section_2, child flange_2_bolts, origin xyz=0 0 0 rpy=0 0 0
- added joint flange_3_bolts_joint: type fixed, parent tower_section_3, child flange_3_bolts, origin xyz=0 0 0 rpy=0 0 0
- added joint tower_inspect_flange_1_joint: type fixed, parent tower_section_1, child tower_inspect_flange_1, origin xyz=2.77203 0 21.446 rpy=0 0 0
- added joint tower_inspect_flange_2_joint: type fixed, parent tower_section_2, child tower_inspect_flange_2, origin xyz=1.39448 2.41531 32.246 rpy=0 0 0
- added joint tower_inspect_flange_3_joint: type fixed, parent tower_section_3, child tower_inspect_flange_3, origin xyz=-3.70381e-16 -2.01626 32.2495 rpy=0 0 0
- joint service_lift_joint: limit lower=0.0 upper=105.66000000000001 effort=100 velocity=4.0 -> lower=-0.1 upper=105.66000000000001 effort=100 velocity=4.0
- joint tower_inspect_cable_loop_joint: origin xyz=0.139 -0.001 19.27 rpy=0 0 0 -> xyz=0.099 0.159 19.27 rpy=0 0 0

File: urdf/scenarios/nacelle_systems_faults.urdf (robot description, URDF)
Before this commit: robot windturbine, 106 links, 105 joints
Links:
- added link flange_1_bolts, mass 1.0; visual mesh filename=package://windturbine_model/models/tower_interior/flange_1_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
- added link flange_2_bolts, mass 1.0; visual mesh filename=package://windturbine_model/models/tower_interior/flange_2_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
- added link flange_3_bolts, mass 1.0; visual mesh filename=package://windturbine_model/models/tower_interior/flange_3_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
- added link tower_inspect_flange_1, mass 1.0
- added link tower_inspect_flange_2, mass 1.0
- added link tower_inspect_flange_3, mass 1.0
Joints:
- added joint flange_1_bolts_joint: type fixed, parent tower_section_1, child flange_1_bolts, origin xyz=0 0 0 rpy=0 0 0
- added joint flange_2_bolts_joint: type fixed, parent tower_section_2, child flange_2_bolts, origin xyz=0 0 0 rpy=0 0 0
- added joint flange_3_bolts_joint: type fixed, parent tower_section_3, child flange_3_bolts, origin xyz=0 0 0 rpy=0 0 0
- added joint tower_inspect_flange_1_joint: type fixed, parent tower_section_1, child tower_inspect_flange_1, origin xyz=2.77203 0 21.446 rpy=0 0 0
- added joint tower_inspect_flange_2_joint: type fixed, parent tower_section_2, child tower_inspect_flange_2, origin xyz=1.39448 2.41531 32.246 rpy=0 0 0
- added joint tower_inspect_flange_3_joint: type fixed, parent tower_section_3, child tower_inspect_flange_3, origin xyz=-3.70381e-16 -2.01626 32.2495 rpy=0 0 0
- joint service_lift_joint: limit lower=0.0 upper=105.66000000000001 effort=100 velocity=4.0 -> lower=-0.1 upper=105.66000000000001 effort=100 velocity=4.0
- joint tower_inspect_cable_loop_joint: origin xyz=0.139 -0.001 19.27 rpy=0 0 0 -> xyz=0.099 0.159 19.27 rpy=0 0 0

File: urdf/scenarios/outside_all_faults.urdf (robot description, URDF)
Before this commit: robot windturbine, 112 links, 111 joints
Links:
- added link flange_1_bolts, mass 1.0; visual mesh filename=package://windturbine_model/models/tower_interior/flange_1_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
- added link flange_2_bolts, mass 1.0; visual mesh filename=package://windturbine_model/models/tower_interior/flange_2_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
- added link flange_3_bolts, mass 1.0; visual mesh filename=package://windturbine_model/models/tower_interior/flange_3_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
- added link tower_inspect_flange_1, mass 1.0
- added link tower_inspect_flange_2, mass 1.0
- added link tower_inspect_flange_3, mass 1.0
Joints:
- added joint flange_1_bolts_joint: type fixed, parent tower_section_1, child flange_1_bolts, origin xyz=0 0 0 rpy=0 0 0
- added joint flange_2_bolts_joint: type fixed, parent tower_section_2, child flange_2_bolts, origin xyz=0 0 0 rpy=0 0 0
- added joint flange_3_bolts_joint: type fixed, parent tower_section_3, child flange_3_bolts, origin xyz=0 0 0 rpy=0 0 0
- added joint tower_inspect_flange_1_joint: type fixed, parent tower_section_1, child tower_inspect_flange_1, origin xyz=2.77203 0 21.446 rpy=0 0 0
- added joint tower_inspect_flange_2_joint: type fixed, parent tower_section_2, child tower_inspect_flange_2, origin xyz=1.39448 2.41531 32.246 rpy=0 0 0
- added joint tower_inspect_flange_3_joint: type fixed, parent tower_section_3, child tower_inspect_flange_3, origin xyz=-3.70381e-16 -2.01626 32.2495 rpy=0 0 0
- joint service_lift_joint: limit lower=0.0 upper=105.66000000000001 effort=100 velocity=4.0 -> lower=-0.1 upper=105.66000000000001 effort=100 velocity=4.0
- joint tower_inspect_cable_loop_joint: origin xyz=0.139 -0.001 19.27 rpy=0 0 0 -> xyz=0.099 0.159 19.27 rpy=0 0 0

File: urdf/scenarios/outside_ground.urdf (robot description, URDF)
Before this commit: robot windturbine, 108 links, 107 joints
Links:
- added link flange_1_bolts, mass 1.0; visual mesh filename=package://windturbine_model/models/tower_interior/flange_1_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
- added link flange_2_bolts, mass 1.0; visual mesh filename=package://windturbine_model/models/tower_interior/flange_2_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
- added link flange_3_bolts, mass 1.0; visual mesh filename=package://windturbine_model/models/tower_interior/flange_3_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
- added link tower_inspect_flange_1, mass 1.0
- added link tower_inspect_flange_2, mass 1.0
- added link tower_inspect_flange_3, mass 1.0
Joints:
- added joint flange_1_bolts_joint: type fixed, parent tower_section_1, child flange_1_bolts, origin xyz=0 0 0 rpy=0 0 0
- added joint flange_2_bolts_joint: type fixed, parent tower_section_2, child flange_2_bolts, origin xyz=0 0 0 rpy=0 0 0
- added joint flange_3_bolts_joint: type fixed, parent tower_section_3, child flange_3_bolts, origin xyz=0 0 0 rpy=0 0 0
- added joint tower_inspect_flange_1_joint: type fixed, parent tower_section_1, child tower_inspect_flange_1, origin xyz=2.77203 0 21.446 rpy=0 0 0
- added joint tower_inspect_flange_2_joint: type fixed, parent tower_section_2, child tower_inspect_flange_2, origin xyz=1.39448 2.41531 32.246 rpy=0 0 0
- added joint tower_inspect_flange_3_joint: type fixed, parent tower_section_3, child tower_inspect_flange_3, origin xyz=-3.70381e-16 -2.01626 32.2495 rpy=0 0 0
- joint service_lift_joint: limit lower=0.0 upper=105.66000000000001 effort=100 velocity=4.0 -> lower=-0.1 upper=105.66000000000001 effort=100 velocity=4.0
- joint tower_inspect_cable_loop_joint: origin xyz=0.139 -0.001 19.27 rpy=0 0 0 -> xyz=0.099 0.159 19.27 rpy=0 0 0

File: urdf/scenarios/tower_bolt_check.urdf (robot description, URDF)
Before this commit: robot windturbine, 113 links, 112 joints
Links:
- removed link generator_fault_carbon_dust
- removed link generator_fault_terminal_heat
- link fast_shaft_brake_disc: geometry collision cylinder length=0.06 radius=0.45; visual mesh filename=package://windturbine_model/models/generator/brake_disc_ok.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
- link fast_shaft_coupling: geometry collision cylinder length=0.55 radius=0.3; visual mesh filename=package://windturbine_model/models/generator/coupling_ok.obj
Joints:
- removed joint generator_fault_carbon_dust_joint
- removed joint generator_fault_terminal_heat_joint

File: urdf/scenarios/tower_climb.urdf (robot description, URDF)
Before this commit: robot windturbine, 106 links, 105 joints
Links:
- added link flange_1_bolts, mass 1.0; visual mesh filename=package://windturbine_model/models/tower_interior/flange_1_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
- added link flange_2_bolts, mass 1.0; visual mesh filename=package://windturbine_model/models/tower_interior/flange_2_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
- added link flange_3_bolts, mass 1.0; visual mesh filename=package://windturbine_model/models/tower_interior/flange_3_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
- added link tower_inspect_flange_1, mass 1.0
- added link tower_inspect_flange_2, mass 1.0
- added link tower_inspect_flange_3, mass 1.0
Joints:
- added joint flange_1_bolts_joint: type fixed, parent tower_section_1, child flange_1_bolts, origin xyz=0 0 0 rpy=0 0 0
- added joint flange_2_bolts_joint: type fixed, parent tower_section_2, child flange_2_bolts, origin xyz=0 0 0 rpy=0 0 0
- added joint flange_3_bolts_joint: type fixed, parent tower_section_3, child flange_3_bolts, origin xyz=0 0 0 rpy=0 0 0
- added joint tower_inspect_flange_1_joint: type fixed, parent tower_section_1, child tower_inspect_flange_1, origin xyz=2.77203 0 21.446 rpy=0 0 0
- added joint tower_inspect_flange_2_joint: type fixed, parent tower_section_2, child tower_inspect_flange_2, origin xyz=1.39448 2.41531 32.246 rpy=0 0 0
- added joint tower_inspect_flange_3_joint: type fixed, parent tower_section_3, child tower_inspect_flange_3, origin xyz=-3.70381e-16 -2.01626 32.2495 rpy=0 0 0
- joint service_lift_joint: limit lower=0.0 upper=105.66000000000001 effort=100 velocity=4.0 -> lower=-0.1 upper=105.66000000000001 effort=100 velocity=4.0
