Commit message: MuJoCo physics replay of the G1 recordings, and the plan flaws it found
scripts/physics_replay.py replays a CRAMERA recording in MuJoCo: turbine collisions
as static (moving links kinematic), the G1 from its URDF with masses, collision
meshes and servos limited to the joint efforts, the pelvis welded to the recorded
path, free objects with mass and friction. It writes a <bundle>_physics bundle and
a report of robot-turbine contacts and carried-object results.

Fixed from its findings:
- plinth collision boxes had zero height (plinth top flush with the ground);
- the bedplate rear frame ran along the floor to the rear wall, across the hoist
  area; it now ends behind the slip ring;
- T3/T4 clipped the tool-rack corner, T5 left the lift car through its railing;
- nacelle walkway: standpoints kept inside the walkway, moves along the walkway
  centre facing along it.

Open: CRAM's G1 grasp puts the palm inside the tool case (the case slips out in
physics); the parked hands barely fit the 0.69 m walkway.

Co-Authored-By: Claude Opus 5.5 <noreply@anthropic.com>
Claude-Session: https://claude.ai/code/session_01BXKsjsesbT14QvbqkbYZ34

File: urdf/scenarios/after_maintenance.urdf (robot description, URDF)
Before this commit: robot windturbine, 111 links, 110 joints
Links:
- link bedplate: geometry collision box size=0.1 0.24 0.693217; collision box size=0.1 0.24 0.693217
- link foundation: geometry collision box size=1.16228 1.04689 0.8; collision box size=1.16228 1.04689 0.8

File: urdf/scenarios/blade_damage.urdf (robot description, URDF)
Before this commit: robot windturbine, 114 links, 113 joints
Links:
- link bedplate: geometry collision box size=0.1 0.24 0.693217; collision box size=0.1 0.24 0.693217
- link foundation: geometry collision box size=1.16228 1.04689 0.8; collision box size=1.16228 1.04689 0.8

File: urdf/scenarios/bring_the_tool.urdf (robot description, URDF)
Before this commit: robot windturbine, 112 links, 111 joints
Links:
- link bedplate: geometry collision box size=0.1 0.24 0.693217; collision box size=0.1 0.24 0.693217
- link foundation: geometry collision box size=1.16228 1.04689 0.8; collision box size=1.16228 1.04689 0.8

File: urdf/scenarios/gearbox_all_faults.urdf (robot description, URDF)
Before this commit: robot windturbine, 113 links, 112 joints
Links:
- link bedplate: geometry collision box size=0.1 0.24 0.693217; collision box size=0.1 0.24 0.693217
- link foundation: geometry collision box size=1.16228 1.04689 0.8; collision box size=1.16228 1.04689 0.8

File: urdf/scenarios/gearbox_seal_leak.urdf (robot description, URDF)
Before this commit: robot windturbine, 113 links, 112 joints
Links:
- link bedplate: geometry collision box size=0.1 0.24 0.693217; collision box size=0.1 0.24 0.693217
- link foundation: geometry collision box size=1.16228 1.04689 0.8; collision box size=1.16228 1.04689 0.8

File: urdf/scenarios/generator_all_faults.urdf (robot description, URDF)
Before this commit: robot windturbine, 113 links, 112 joints
Links:
- link bedplate: geometry collision box size=0.1 0.24 0.693217; collision box size=0.1 0.24 0.693217
- link foundation: geometry collision box size=1.16228 1.04689 0.8; collision box size=1.16228 1.04689 0.8

File: urdf/scenarios/hoist_access.urdf (robot description, URDF)
Before this commit: robot windturbine, 111 links, 110 joints
Links:
- link bedplate: geometry collision box size=0.1 0.24 0.693217; collision box size=0.1 0.24 0.693217
- link foundation: geometry collision box size=1.16228 1.04689 0.8; collision box size=1.16228 1.04689 0.8

File: urdf/scenarios/main_shaft_all_faults.urdf (robot description, URDF)
Before this commit: robot windturbine, 113 links, 112 joints
Links:
- link bedplate: geometry collision box size=0.1 0.24 0.693217; collision box size=0.1 0.24 0.693217
- link foundation: geometry collision box size=1.16228 1.04689 0.8; collision box size=1.16228 1.04689 0.8

File: urdf/scenarios/nacelle_all_faults.urdf (robot description, URDF)
Before this commit: robot windturbine, 118 links, 117 joints
Links:
- link bedplate: geometry collision box size=0.1 0.24 0.693217; collision box size=0.1 0.24 0.693217
- link foundation: geometry collision box size=1.16228 1.04689 0.8; collision box size=1.16228 1.04689 0.8

File: urdf/scenarios/nacelle_systems_faults.urdf (robot description, URDF)
Before this commit: robot windturbine, 112 links, 111 joints
Links:
- link bedplate: geometry collision box size=0.1 0.24 0.693217; collision box size=0.1 0.24 0.693217
- link foundation: geometry collision box size=1.16228 1.04689 0.8; collision box size=1.16228 1.04689 0.8

File: urdf/scenarios/outside_all_faults.urdf (robot description, URDF)
Before this commit: robot windturbine, 118 links, 117 joints
Links:
- link bedplate: geometry collision box size=0.1 0.24 0.693217; collision box size=0.1 0.24 0.693217
- link foundation: geometry collision box size=1.16228 1.04689 0.8; collision box size=1.16228 1.04689 0.8

File: urdf/scenarios/outside_ground.urdf (robot description, URDF)
Before this commit: robot windturbine, 114 links, 113 joints
Links:
- link bedplate: geometry collision box size=0.1 0.24 0.693217; collision box size=0.1 0.24 0.693217
- link foundation: geometry collision box size=1.16228 1.04689 0.8; collision box size=1.16228 1.04689 0.8

File: urdf/scenarios/tower_bolt_check.urdf (robot description, URDF)
Before this commit: robot windturbine, 111 links, 110 joints
Links:
- link bedplate: geometry collision box size=0.1 0.24 0.693217; collision box size=0.1 0.24 0.693217
- link foundation: geometry collision box size=1.16228 1.04689 0.8; collision box size=1.16228 1.04689 0.8

File: urdf/scenarios/tower_climb.urdf (robot description, URDF)
Before this commit: robot windturbine, 112 links, 111 joints
Links:
- link bedplate: geometry collision box size=0.1 0.24 0.693217; collision box size=0.1 0.24 0.693217
- link foundation: geometry collision box size=1.16228 1.04689 0.8; collision box size=1.16228 1.04689 0.8
